File: circuit/emi-board.kicad_pcb (KiCad board)
At the start: 2 copper layers, 40.5 x 52.5 mm, 8 parts, among them J1 EMI-MAIN

Commit message: PCB 작업
Parts:
- J1: footprint Connector_JST:JST_PH_B2B-PH-K_1x02_P2.00mm_Vertical -> Connector_Coaxial:U.FL_Hirose_U.FL-R-SMT-1_Vertical
- moved C2A1 3.61 mm to (157.5, 79.0), turned to -90 degrees
- moved R1 0.74 mm to (164.0, 82.5)
- moved C1 0.56 mm to (152.2, 81.5)
- turned J1 to 180 degrees
Connections:
- C1 pad 1: Net-(J1-GND) -> Net-(J1-EMI_SIG)
- C1 pad 2: Net-(C1-Pad2) -> Net-(J1-EMI_SIG)
- C2A1 pad 1: Net-(C2A1-Pad1) -> Net-(J1-EMI_SIG)
- C2A1 pad 2: Net-(C1-Pad2) -> Net-(J1-EMI_SIG)
- J1 pad 2: Net-(J1-GND) -> Net-(J1-EMI_SIG)
- R1 pad 1: Net-(C2A1-Pad1) -> Net-(J1-EMI_SIG)
- R1 pad 2: Net-(L1-Pad2) -> Net-(J1-EMI_SIG)
Routing:
- net Net-(J1-EMI_SIG): track 46.6 -> 49.7 mm
