File: circuit/emi-board.kicad_sch (KiCad schematic)
At the start: 5 parts, among them J1 EMI-MAIN

Commit message: PCB 작업
Parts:
- J1: footprint Connector_JST:JST_PH_B2B-PH-K_1x02_P2.00mm_Vertical -> Connector_Coaxial:U.FL_Hirose_U.FL-R-SMT-1_Vertical
Connections:
- net at J1.1 (EMI_SIG), L1.1: now also C1.2, C2A1.1
- net at C1.1, J1.2 (GND): now also C2A1.2, R1.1
Other:
- moved on the sheet: C1, C2A1, R1
Changed lines of the file:
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@@
 	(generator_version "9.0")
 	(paper "A4")
-	(wire
-		(pts
-			(xy 121.92 93.98) (xy 168.91 93.98)
-		)
-		(stroke
-			(width 0)
-			(type default)
-		)
-	)
-	(wire
-		(pts
-			(xy 176.53 93.98) (xy 176.53 107.95)
-		)
-		(stroke
-			(width 0)
-			(type default)
-		)
-	)
-	(wire
-		(pts
-			(xy 128.27 107.95) (xy 128.27 96.52)
-		)
-		(stroke
-			(width 0)
-			(type default)
-		)
-	)
-	(wire
-		(pts
-			(xy 143.51 107.95) (xy 151.13 107.95)
-		)
-		(stroke
-			(width 0)
-			(type default)
-		)
-	)
-	(wire
-		(pts
-			(xy 158.75 107.95) (xy 168.91 107.95)
-		)
-		(stroke
-			(width 0)
-			(type default)
-		)
-	)
-	(wire
-		(pts
-			(xy 135.89 107.95) (xy 128.27 107.95)
-		)
-		(stroke
-			(width 0)
-			(type default)
-		)
-	)
-	(wire
-		(pts
-			(xy 128.27 96.52) (xy 121.92 96.52)
+	(junction
+		(at 140.97 101.6)
+		(diameter 0)
+		(color 0 0 0 0)
+	)
+	(junction
+		(at 156.21 101.6)
+		(diameter 0)
+		(color 0 0 0 0)
+	)
+	(junction
+		(at 140.97 93.98)
+		(diameter 0)
+		(color 0 0 0 0)
+	)
+	(junction
+		(at 156.21 93.98)
+		(diameter 0)
+		(color 0 0 0 0)
+	)
+	(wire
+		(pts
+			(xy 121.92 93.98) (xy 140.97 93.98)
+		)
+		(stroke
+			(width 0)
+			(type default)
+		)
+	)
+	(wire
+		(pts
+			(xy 176.53 93.98) (xy 176.53 101.6)
+		)
+		(stroke
+			(width 0)
+			(type default)
+		)
+	)
+	(wire
+		(pts
+			(xy 133.35 101.6) (xy 133.35 96.52)
+		)
+		(stroke
+			(width 0)
+			(type default)
+		)
+	)
+	(wire
+		(pts
+			(xy 140.97 101.6) (xy 156.21 101.6)
+		)
+		(stroke
+			(width 0)
+			(type default)
+		)
+	)
+	(wire
+		(pts
+			(xy 156.21 101.6) (xy 168.91 101.6)
+		)
+		(stroke
+			(width 0)
+			(type default)
+		)
+	)
+	(wire
+		(pts
+			(xy 156.21 93.98) (xy 168.91 93.98)
+		)
+		(stroke
+			(width 0)
+			(type default)
+		)
+	)
+	(wire
+		(pts
+			(xy 140.97 101.6) (xy 133.35 101.6)
+		)
+		(stroke
+			(width 0)
+			(type default)
+		)
+	)
+	(wire
+		(pts
+			(xy 140.97 93.98) (xy 156.21 93.98)
+		)
+		(stroke
+			(width 0)
+			(type default)
+		)
+	)
+	(wire
+		(pts
+			(xy 133.35 96.52) (xy 121.92 96.52)
 		)
 		(stroke
@@
 			)
 		)
-		(property "Footprint" "Connector_JST:JST_PH_B2B-PH-K_1x02_P2.00mm_Vertical"
+		(property "Footprint" "Connector_Coaxial:U.FL_Hirose_U.FL-R-SMT-1_Vertical"
 			(at 116.84 93.98 0)
 			(effects
@@
 	(symbol
 		(lib_id "Device:C")
-		(at 139.7 107.95 90)
+		(at 140.97 97.79 0)
 		(mirror x)
 		(unit 1)
@@
 		(dnp no)
 		(property "Reference" "C1"
-			(at 138.4299 111.76 0)
+			(at 144.78 99.0601 0)
 			(effects
 				(font
@@
 		)
 		(property "Value" "0.01uF"
-			(at 140.9699 111.76 0)
+			(at 144.78 96.5201 0)
 			(effects
 				(font
@@
 		)
 		(property "Footprint" "Capacitor_THT:C_Disc_D5.0mm_W2.5mm_P2.50mm"
-			(at 143.51 108.9152 0)
+			(at 141.9352 93.98 0)
 			(effects
 				(font
@@
 		)
 		(property "Datasheet" "~"
-			(at 139.7 107.95 0)
+			(at 140.97 97.79 0)
 			(effects
 				(font
@@
 		)
 		(property "Description" "Unpolarized capacitor"
-			(at 139.7 107.95 0)
+			(at 140.97 97.79 0)
 			(effects
 				(font
@@
 	(symbol
 		(lib_id "Device:R")
-		(at 172.72 107.95 90)
+		(at 172.72 101.6 90)
 		(unit 1)
 		(exclude_from_sim no)
@@
 		(on_board yes)
 		(dnp no)
-		(fields_autoplaced yes)
 		(property "Reference" "R1"
-			(at 172.72 101.6 90)
+			(at 172.974 103.886 90)
 			(effects
 				(font
@@
 		)
 		(property "Value" "100k"
-			(at 172.72 104.14 90)
+			(at 172.974 106.426 90)
 			(effects
 				(font
@@
 		)
 		(property "Footprint" "Resistor_THT:R_Axial_DIN0204_L3.6mm_D1.6mm_P5.08mm_Horizontal"
-			(at 172.72 109.728 90)
+			(at 172.72 103.378 90)
 			(effects
 				(font
@@
 		)
 		(property "Datasheet" "~"
-			(at 172.72 107.95 0)
+			(at 172.72 101.6 0)
 			(effects
 				(font
@@
 		)
 		(property "Description" "Resistor"
-			(at 172.72 107.95 0)
+			(at 172.72 101.6 0)
 			(effects
 				(font
@@
 	(symbol
 		(lib_id "Device:C")
-		(at 154.94 107.95 270)
-		(mirror x)
+		(at 156.21 97.79 0)
+		(mirror y)
 		(unit 1)
 		(exclude_from_sim no)
@@
 		(dnp no)
 		(property "Reference" "C2A1"
-			(at 154.94 115.57 90)
+			(at 163.83 97.79 90)
 			(effects
 				(font
@@
 		)
 		(property "Value" "DNP"
-			(at 154.94 113.03 90)
+			(at 161.29 97.79 90)
 			(effects
 				(font
@@
 		)
 		(property "Footprint" "Capacitor_THT:C_Disc_D5.0mm_W2.5mm_P2.50mm"
-			(at 151.13 106.9848 0)
+			(at 155.2448 101.6 0)
 			(effects
 				(font
@@
 		)
 		(property "Datasheet" "~"
-			(at 154.94 107.95 0)
+			(at 156.21 97.79 0)
 			(effects
 				(font
@@
 		)
 		(property "Description" "Unpolarized capacitor"
-			(at 154.94 107.95 0)
-			(effects
-				(font
+			(at 156.21 97.79 0)
+			(effects
+				(font
