File: circuit/main-board.kicad_sch (KiCad schematic)
At the start: 14 parts, among them J1 EMI-MAIN, J2 Conn_01x08, J3 LED-line-socket, J4 Conn_01x08, J5 DHT22_Conn_3Pin, Q1 2N2222

Commit message: PCB 작업
Parts:
- J1: footprint Connector_JST:JST_PH_B2B-PH-K_1x02_P2.00mm_Vertical -> Connector_Coaxial:U.FL_Hirose_U.FL-R-SMT-1_Vertical
Changed lines of the file:
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@@
 			)
 		)
-		(property "Footprint" "Connector_JST:JST_PH_B2B-PH-K_1x02_P2.00mm_Vertical"
+		(property "Footprint" "Connector_Coaxial:U.FL_Hirose_U.FL-R-SMT-1_Vertical"
 			(at 68.58 69.85 0)
 			(effects
