File: circuit/main-board.kicad_pcb (KiCad board)
At the start: 4 copper layers, 40.5 x 52.5 mm, 18 parts, among them J1 EMI-MAIN, J2 Conn_01x08, J3 LED-line-socket, J4 Conn_01x08, J5 DHT22_Conn_3Pin, Q1 2N2222

Commit message: PCB 작업
Parts:
- J1: footprint Connector_JST:JST_PH_B2B-PH-K_1x02_P2.00mm_Vertical -> Connector_Coaxial:U.FL_Hirose_U.FL-R-SMT-1_Vertical
Routing:
- net GND: track 0.00 -> 90.2 mm
- net Net-(J4-Pin_8): track 0.00 -> 39.4 mm
- net Net-(J2-Pin_2): track 0.00 -> 26.1 mm
- net Net-(Q1-B): track 0.00 -> 20.9 mm
- net Net-(J2-Pin_5): track 0.00 -> 19.8 mm
- net Net-(J2-Pin_6): track 0.00 -> 18.5 mm
- net Net-(J4-Pin_3): track 0.00 -> 16.1 mm
- net Net-(D1-K1): track 0.00 -> 15.5 mm
- net Net-(J3-IR_LED-): track 0.00 -> 14.5 mm
- net Net-(J3-IR_LED+): track 0.00 -> 10.5 mm
- net Net-(D1-K2): track 0.00 -> 9.66 mm
- net Net-(J2-Pin_4): track 0.00 -> 8.42 mm

Commit message: PCB 작업
Routing:
- net Net-(J1-EMI_SIG): track 0.00 -> 23.9 mm
- net Net-(J3-IR_LED-): track 14.5 -> 16.2 mm
- net GND: track 90.2 -> 89.7 mm
- removed copper zone on In1.Cu, net GND
Changed lines of the file:
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@@
 		(pcbplotparams
 			(layerselection 0x00000000_00000000_55555555_5755f5ff)
-			(plot_on_all_layers_selection 0x00000000_00000000_00000000_020000af)
+			(plot_on_all_layers_selection 0x00000000_00000000_00000000_00000000)
 			(disableapertmacros no)
 			(usegerberextensions no)
@@
 		(layer "Edge.Cuts")
 	)
-	(gr_text "TX\nRX\nD1\nD2\nD3\nD4\nGND\n5V\n"
-		(at 159 114.75 0)
-		(layer "F.Cu")
-		(effects
-			(font
-				(size 1 1)
-				(thickness 0.15)
-			)
-			(justify left bottom)
-		)
-	)
 	(gr_text "+"
 		(at 150.985 81.25 0)
@@
 		)
 	)
+	(gr_text "TX\nRX\nD1\nD2\nD3\nD4\nGND\n5V\n"
+		(at 159 114.75 0)
+		(layer "F.SilkS")
+		(effects
+			(font
+				(size 1 1)
+				(thickness 0.15)
+			)
+			(justify left bottom)
+		)
+	)
 	(gr_text "E"
 		(at 149 85 0)
@@
 	)
 	(segment
-		(start 136.025 79.225)
-		(end 139.5 82.7)
+		(start 145.46 97.29)
+		(end 145.25 97.5)
+		(width 0.2)
+		(layer "F.Cu")
+		(net 2)
+	)
+	(segment
+		(start 132.75 85.5)
+		(end 139.25 85.5)
+		(width 0.2)
+		(layer "F.Cu")
+		(net 2)
+	)
+	(segment
+		(start 145.25 92)
+		(end 145.46 92.21)
+		(width 0.2)
+		(layer "F.Cu")
+		(net 2)
+	)
+	(segment
+		(start 145.46 96.75)
+		(end 145.46 97.29)
+		(width 0.2)
+		(layer "F.Cu")
+		(net 2)
+	)
+	(segment
+		(start 149.25 103)
+		(end 149.25 105)
 		(width 0.2)
 		(layer "B.Cu")
@@
 	)
 	(segment
-		(start 139.5 82.7)
-		(end 139.5 85.25)
+		(start 145.46 96.75)
+		(end 145.46 99.21)
 		(width 0.2)
 		(layer "B.Cu")
@@
 		(end 162 113.25)
 		(width 0.2)
-		(layer "In2.Cu")
+		(layer "B.Cu")
 		(net 2)
 	)
 	(segment
-		(start 145.46 107.296372)
-		(end 145.46 96.75)
+		(start 145.25 91)
+		(end 145.25 92)
 		(width 0.2)
-		(layer "In2.Cu")
+		(layer "B.Cu")
 		(net 2)
 	)
 	(segment
-		(start 145.46 91.21)
-		(end 145.46 96.75)
+		(start 139.5 85.25)
+		(end 145.25 91)
 		(width 0.2)
-		(layer "In2.Cu")
+		(layer "B.Cu")
 		(net 2)
 	)
 	(segment
-		(start 156.46 118.296372)
-		(end 145.46 107.296372)
+		(start 145.46 99.21)
+		(end 149.25 103)
 		(width 0.2)
-		(layer "In2.Cu")
+		(layer "B.Cu")
 		(net 2)
 	)
 	(segment
-		(start 139.5 85.25)
-		(end 145.46 91.21)
+		(start 136.025 79.225)
+		(end 139.5 82.7)
 		(width 0.2)
-		(layer "In2.Cu")
+		(layer "B.Cu")
+		(net 2)
+	)
+	(segment
+		(start 153.96 118.79)
+		(end 156.46 118.79)
+		(width 0.2)
+		(layer "B.Cu")
+		(net 2)
+	)
+	(segment
+		(start 153.75 118.58)
+		(end 153.96 118.79)
+		(width 0.2)
+		(layer "B.Cu")
+		(net 2)
+	)
+	(segment
+		(start 139.5 82.7)
+		(end 139.5 85.25)
+		(width 0.2)
+		(layer "B.Cu")
+		(net 2)
+	)
+	(segment
+		(start 145.46 92.21)
+		(end 145.46 96.75)
+		(width 0.2)
+		(layer "B.Cu")
 		(net 2)
 	)
@@
 		(end 162 97.33)
 		(width 0.2)
-		(layer "In2.Cu")
+		(layer "B.Cu")
 		(net 2)
 	)
 	(segment
-		(start 132.75 85.5)
-		(end 139.25 85.5)
+		(start 149.25 105)
+		(end 151.75 107.5)
 		(width 0.2)
-		(layer "In2.Cu")
+		(layer "B.Cu")
 		(net 2)
 	)
 	(segment
-		(start 156.46 118.79)
-		(end 156.46 118.296372)
+		(start 151.75 107.5)
+		(end 153.75 107.5)
 		(width 0.2)
-		(layer "In2.Cu")
+		(layer "B.Cu")
 		(net 2)
 	)
@@
 		(end 145.46 92.25)
 		(width 0.2)
-		(layer "In2.Cu")
+		(layer "B.Cu")
 		(net 2)
 	)
 	(segment
-		(start 139.25 85.5)
-		(end 139.5 85.25)
+		(start 153.75 107.5)
+		(end 153.75 118.58)
 		(width 0.2)
-		(layer "In2.Cu")
+		(layer "B.Cu")
 		(net 2)
 	)
 	(segment
-		(start 145.46 92.25)
-		(end 145.46 96.75)
+		(start 156.46 118.79)
+		(end 156.46 118.296372)
 		(width 0.2)
 		(layer "In2.Cu")
@@
 	)
 	(segment
-		(start 146.92 104.75)
-		(end 135.42 116.25)
+		(start 139.25 85.5)
+		(end 139.5 85.25)
 		(width 0.2)
-		(layer "B.Cu")
-		(net 4)
+		(layer "In2.Cu")
+		(net 2)
 	)
 	(segment
@@
 	(segment
 		(start 146.92 104.75)
+		(end 135.42 116.25)
+		(width 0.2)
+		(layer "In1.Cu")
+		(net 4)
+	)
+	(segment
+		(start 146.92 104.75)
 		(end 147 104.75)
 		(width 0.2)
@@
 		(end 163.151 93.401)
 		(width 0.2)
-		(layer "In2.Cu")
+		(layer "F.Cu")
 		(net 14)
 	)
@@
 		(end 163.151 114.639)
 		(width 0.2)
-		(layer "In2.Cu")
+		(layer "F.Cu")
 		(net 14)
 	)
@@
 		(end 163.29 90.96)
 		(width 0.2)
-		(layer "In2.Cu")
+		(layer "F.Cu")
 		(net 14)
 	)
@@
 		(end 156.46 121.33)
 		(width 0.2)
-		(layer "In2.Cu")
+		(layer "F.Cu")
 		(net 14)
 	)
@@
 		(end 162 92.25)
 		(width 0.2)
-		(layer "In2.Cu")
+		(layer "F.Cu")
 		(net 14)
 	)
@@
 		(end 151.73 87.25)
 		(width 0.2)
-		(layer "B.Cu")
+		(layer "In1.Cu")
 		(net 17)
 	)
@@
 		(end 151.73 96.52)
 		(width 0.2)
-		(layer "B.Cu")
+		(layer "In1.Cu")
 		(net 17)
 	)
 	(segment
-		(start 152.599 86.849)
-		(end 153 87.25)
+		(start 154.324 76.074)
+		(end 155.5 77.25)
 		(width 0.2)
-		(layer "In2.Cu")
+		(layer "F.Cu")
 		(net 18)
 	)
@@
 		(end 152.91484 76.074)
 		(width 0.2)
-		(layer "In2.Cu")
+		(layer "F.Cu")
+		(net 18)
+	)
+	(segment
+		(start 152.91484 76.074)
+		(end 152.599 76.38984)
+		(width 0.2)
+		(layer "F.Cu")
+		(net 18)
+	)
+	(segment
+		(start 152.599 76.38984)
+		(end 152.599 86.849)
+		(width 0.2)
+		(layer "F.Cu")
 		(net 18)
 	)
@@
 		(end 154.324 76.074)
 		(width 0.2)
-		(layer "In2.Cu")
+		(layer "In1.Cu")
 		(net 18)
 	)
 	(segment
-		(start 152.91484 76.074)
-		(end 152.599 76.38984)
+		(start 152.599 86.849)
+		(end 153 87.25)
 		(width 0.2)
 		(layer "In2.Cu")
@@
 	)
 	(segment
-		(start 152.599 76.38984)
-		(end 152.599 86.849)
+		(start 134.624 89.124)
+		(end 138.5 93)
 		(width 0.2)
-		(layer "In2.Cu")
-		(net 18)
+		(layer "B.Cu")
+		(net 19)
+	)
+	(segment
+		(start 137.11016 75.449)
+		(end 134.93984 75.449)
+		(width 0.2)
+		(layer "B.Cu")
+		(net 19)
+	)
+	(segment
+		(start 134.624 75.76484)
+		(end 134.624 89.124)
+		(width 0.2)
+		(layer "B.Cu")
+		(net 19)
+	)
+	(segment
+		(start 137.55 77.75)
+		(end 137.55 75.88884)
+		(width 0.2)
+		(layer "B.Cu")
+		(net 19)
+	)
+	(segment
+		(start 137.55 75.88884)
+		(end 137.11016 75.449)
+		(width 0.2)
+		(layer "B.Cu")
+		(net 19)
+	)
+	(segment
+		(start 134.93984 75.449)
+		(end 134.624 75.76484)
+		(width 0.2)
+		(layer "B.Cu")
+		(net 19)
 	)
 	(segment
@@
 		(end 158.21 85.75)
 		(width 0.2)
-		(layer "In2.Cu")
+		(layer "F.Cu")
 		(net 20)
 	)
@@
 		(end 153.5 81.04)
 		(width 0.2)
-		(layer "In2.Cu")
+		(layer "F.Cu")
 		(net 20)
 	)
@@
 		(end 152 104.75)
 		(width 0.2)
-		(layer "In2.Cu")
+		(layer "F.Cu")
 		(net 22)
 	)
@@
 		(end 152 100.75)
 		(width 0.2)
-		(layer "In2.Cu")
+		(layer "F.Cu")
 		(net 22)
 	)
@@
 		(net 2)
 		(net_name "GND")
-		(layer "In1.Cu")
-		(hatch edge 0.5)
-		(connect_pads
-			(clearance 0.2)
-		)
-		(min_thickness 0.25)
-		(filled_areas_thickness no)
-		(fill yes
-			(thermal_gap 0.5)
-			(thermal_bridge_width 0.5)
-		)
-		(polygon
-			(pts
-				(xy 121.25 69.5) (xy 121.25 131) (xy 169.75 130.5) (xy 167.25 68)
-			)
-		)
-	)
-	(zone
-		(net 2)
-		(net_name "GND")
 		(layer "In2.Cu")
 		(hatch edge 0.5)
-		(priority 1)
 		(connect_pads
 			(clearance 0.2)
@@
 		(polygon
 			(pts
-				(xy 118.75 68.5) (xy 119.25 134) (xy 178.25 133) (xy 173.25 62.5)
+				(xy 115.75 57.5) (xy 115.75 138.5) (xy 169.25 139) (xy 166.75 60)
 			)
 		)
